File: wimos-pcb-desgin/WIMOS-motherboard.sch (EAGLE design)
At the start: 32 parts

Commit message: Placa de circuito impreso
Parts:
- removed GPIO_A1, GPIO_A2, GPIO_A3, GPIO_A4, GPIO_A5, GPIO_A6: (no value), pinhead:PINHD-1X4/90
- added GPIO_A1_1B, GPIO_A2_1B, GPIO_A3_1B, GPIO_A4_1B: (no value), pinhead:PINHD-1X3/90
- added GPIO_A1_3B: (no value), pinhead:PINHD-1X5/90
- added IC1: 7805T, linear:7805T
- added SERIE_MODULE: (no value), pinhead:PINHD-1X4/90
- GPIO_D1_1B, GPIO_D2_1B, GPIO_D3_1B, GPIO_D4_1B, GPIO_DAC0, GPIO_DAC1: device pinhead:PINHD-1X4/90 -> pinhead:PINHD-1X3/90
- GPIO_D1_2B, GPIO_D2_2B: device pinhead:PINHD-1X5/90 -> pinhead:PINHD-1X4/90
- GPIO_D1_3B, GPIO_D2_3B: device pinhead:PINHD-1X6/90 -> pinhead:PINHD-1X5/90
- GPIO_D1_4B: device pinhead:PINHD-1X7/90 -> pinhead:PINHD-1X6/90
- I2C_MODULE: device pinhead:PINHD-1X4 -> pinhead:PINHD-1X4/90
- POWER_MODULE: device pinhead:PINHD-1X2 -> con-jack:DCJ0303
Connections:
- removed net DUE_PIN26: DUE_MODULE4.8
- removed net GPIO_3.3V: GPIO_A1.1, GPIO_A2.1, GPIO_A3.1, GPIO_A4.1, GPIO_A5.1, GPIO_A6.1, GPIO_D1_1B.1, GPIO_D1_2B.1, GPIO_D1_3B.1, GPIO_D1_4B.1, GPIO_D2_1B.1, GPIO_D2_2B.1, GPIO_D2_3B.1, GPIO_D3_1B.1, GPIO_D4_1B.1, GPIO_DAC0.1, GPIO_DAC1.1
- removed net GPIO_5V: GPIO_A1.2, GPIO_A2.2, GPIO_A3.2, GPIO_A4.2, GPIO_A5.2, GPIO_A6.2, GPIO_D1_1B.2, GPIO_D1_2B.2, GPIO_D1_3B.2, GPIO_D1_4B.2, GPIO_D2_1B.2, GPIO_D2_2B.2, GPIO_D2_3B.2, GPIO_D3_1B.2, GPIO_D4_1B.2, GPIO_DAC0.2, GPIO_DAC1.2
- removed net GPIO_A1: GPIO_A1.3
- removed net GPIO_A2: GPIO_A2.3
- removed net GPIO_A3: GPIO_A3.3
- removed net GPIO_A4: GPIO_A4.3
- removed net GPIO_A5: GPIO_A5.3
- removed net GPIO_A6: GPIO_A6.3
- removed net GPIO_D1_1B: GPIO_D1_1B.3
- removed net GPIO_D1_2.1B: GPIO_D1_2B.3
- removed net GPIO_D1_2.2B: GPIO_D1_2B.4
- removed net GPIO_D1_3.1B: GPIO_D1_3B.3
- removed net GPIO_D1_3.2B: GPIO_D1_3B.4
- removed net GPIO_D1_3.3B: GPIO_D1_3B.5
- removed net GPIO_D1_4.1B: GPIO_D1_4B.3
- removed net GPIO_D1_4.2B: GPIO_D1_4B.4
- removed net GPIO_D1_4.3B: GPIO_D1_4B.5
- removed net GPIO_D1_4.4B: GPIO_D1_4B.6
- removed net GPIO_D2_1B: GPIO_D2_1B.3
- removed net GPIO_D2_2.1B: GPIO_D2_2B.3
- removed net GPIO_D2_2.2B: GPIO_D2_2B.4
- removed net GPIO_D2_3.1B: GPIO_D2_3B.3
- removed net GPIO_D2_3.2B: GPIO_D2_3B.4
- removed net GPIO_D2_3.3B: GPIO_D2_3B.5
- removed net GPIO_D3_1B: GPIO_D3_1B.3
- removed net GPIO_D4_1B: GPIO_D4_1B.3
- removed net GPIO_DAC0: GPIO_DAC0.3
- removed net GPIO_DAC1: GPIO_DAC1.3
- removed net I2C_VCC: CONFIGURATION_MODULE.1, I2C_MODULE.1
- removed net POWER_VCC: POWER_MODULE.1
- new net 5V: CONFIGURATION_MODULE.1, GPIO_A1_1B.2, GPIO_A1_3B.2, GPIO_A2_1B.2, GPIO_A3_1B.2, GPIO_A4_1B.2, GPIO_D1_1B.2, GPIO_D1_2B.2, GPIO_D1_3B.2, GPIO_D1_4B.2, GPIO_D2_1B.2, GPIO_D2_2B.2, GPIO_D2_3B.2, GPIO_D3_1B.2, GPIO_D4_1B.2, GPIO_DAC0.2, GPIO_DAC1.2, I2C_MODULE.1, IC1.VO, SD_MODULE.8
- new net <NONE>: DUE_MODULE1.7
- new net DUE_PIN21: DUE_MODULE4.4
- new net SERIE_RX: SERIE_MODULE.4
- new net SERIE_TX: SERIE_MODULE.3
- new net SERIE_VCC: SERIE_MODULE.1
- new net VCC: IC1.VI, POWER_MODULE.1
- net DUE_5V: no longer SD_MODULE.8
- net DUE_A_PIN_1: now also GPIO_A1_1B.3
- net DUE_A_PIN_10: now also GPIO_A1_3B.3
- net DUE_A_PIN_2: now also GPIO_A2_1B.3
- net DUE_A_PIN_3: now also GPIO_A3_1B.3
- net DUE_A_PIN_4: now also GPIO_A4_1B.3
- net DUE_A_PIN_8: now also GPIO_A1_3B.5
- net DUE_A_PIN_9: now also GPIO_A1_3B.4
- net DUE_DAC0: now also GPIO_DAC0.3
- net DUE_DAC1: now also GPIO_DAC1.3
- net DUE_PIN2: now also GPIO_D2_2B.4
- net DUE_PIN22: now also DUE_MODULE4.3; no longer DUE_MODULE4.4
- net DUE_PIN23: now also DUE_MODULE4.6; no longer DUE_MODULE4.3
- net DUE_PIN24: now also DUE_MODULE4.5; no longer DUE_MODULE4.6
- net DUE_PIN25: now also DUE_MODULE4.7; no longer DUE_MODULE4.5
- net DUE_PIN27: now also DUE_MODULE4.8; no longer DUE_MODULE4.7
- net DUE_PIN28: now also DUE_MODULE4.9; no longer DUE_MODULE4.10
- net DUE_PIN29: now also DUE_MODULE4.10; no longer DUE_MODULE4.9
- net DUE_PIN3: now also GPIO_D2_2B.3
- net DUE_PIN30: now also DUE_MODULE4.11; no longer DUE_MODULE4.12
- net DUE_PIN31: now also DUE_MODULE4.12; no longer DUE_MODULE4.11
- net DUE_PIN32: now also DUE_MODULE4.13; no longer DUE_MODULE4.14
- net DUE_PIN33: now also DUE_MODULE4.14; no longer DUE_MODULE4.13
- net DUE_PIN34: now also DUE_MODULE4.15; no longer DUE_MODULE4.16
- net DUE_PIN35: now also DUE_MODULE4.16, GPIO_D1_3B.3; no longer DUE_MODULE4.15
- net DUE_PIN36: now also DUE_MODULE4.17; no longer DUE_MODULE4.18
- net DUE_PIN37: now also DUE_MODULE4.18, GPIO_D1_3B.4; no longer DUE_MODULE4.17
- net DUE_PIN38: now also DUE_MODULE4.19; no longer DUE_MODULE4.20
- net DUE_PIN39: now also DUE_MODULE4.20, GPIO_D1_3B.5; no longer DUE_MODULE4.19
- net DUE_PIN4: now also GPIO_D1_2B.4
- net DUE_PIN40: now also DUE_MODULE4.21; no longer DUE_MODULE4.22
- net DUE_PIN41: now also DUE_MODULE4.22, GPIO_D2_3B.3; no longer DUE_MODULE4.21
- net DUE_PIN42: now also DUE_MODULE4.23; no longer DUE_MODULE4.24
- net DUE_PIN43: now also DUE_MODULE4.24, GPIO_D2_3B.4; no longer DUE_MODULE4.23
- net DUE_PIN44: now also DUE_MODULE4.25; no longer DUE_MODULE4.26
- net DUE_PIN45: now also DUE_MODULE4.26, GPIO_D2_3B.5; no longer DUE_MODULE4.25
- net DUE_PIN46: now also DUE_MODULE4.27; no longer DUE_MODULE4.28
- net DUE_PIN47: now also DUE_MODULE4.28, GPIO_D1_4B.3; no longer DUE_MODULE4.27
- net DUE_PIN48: now also DUE_MODULE4.29; no longer DUE_MODULE4.30
- net DUE_PIN49: now also DUE_MODULE4.30, GPIO_D1_4B.4; no longer DUE_MODULE4.29
- net DUE_PIN5: now also GPIO_D1_2B.3
- net DUE_PIN50: now also DUE_MODULE4.31; no longer DUE_MODULE4.32
- net DUE_PIN51: now also DUE_MODULE4.32, GPIO_D1_4B.5; no longer DUE_MODULE4.31
- net DUE_PIN52: now also DUE_MODULE4.33; no longer DUE_MODULE4.34
- net DUE_PIN53: now also DUE_MODULE4.34, GPIO_D1_4B.6; no longer DUE_MODULE4.33
- net DUE_PIN6: now also GPIO_D4_1B.3
- net DUE_PIN7: now also GPIO_D3_1B.3
- net DUE_PIN8: now also GPIO_D2_1B.3
- net DUE_PIN9: now also GPIO_D1_1B.3
- net GND: now also GPIO_A1_1B.1, GPIO_A1_3B.1, GPIO_A2_1B.1, GPIO_A3_1B.1, GPIO_A4_1B.1, GPIO_D1_1B.1, GPIO_D1_2B.1, GPIO_D1_3B.1, GPIO_D1_4B.1, GPIO_D2_1B.1, GPIO_D2_2B.1, GPIO_D2_3B.1, GPIO_D3_1B.1, GPIO_D4_1B.1, GPIO_DAC0.1, GPIO_DAC1.1, IC1.GND, POWER_MODULE.3, SERIE_MODULE.2; no longer DUE_MODULE1.7, GPIO_A1.4, GPIO_A2.4, GPIO_A3.4, GPIO_A4.4, GPIO_A5.4, GPIO_A6.4, GPIO_D1_1B.4, GPIO_D1_2B.5, GPIO_D1_3B.6, GPIO_D1_4B.7, GPIO_D2_1B.4, GPIO_D2_2B.5, GPIO_D2_3B.6, GPIO_D3_1B.4, GPIO_D4_1B.4, GPIO_DAC0.4, GPIO_DAC1.4
Other:
- moved on the sheet: CONFIGURATION_MODULE, I2C_MODULE
